Commit message: remove material tags

File: schunk_egp40_description/urdf/schunk_egp40.xacro (robot description, xacro)
@@ -17,13 +17,4 @@
         <xacro:property name="pincer_length" value="0.040" />
         <xacro:property name="pincer_width" value="0.016" />
-        <material name="blue">
-            <color rgba="0 0.2 1 1" />
-        </material>
-        <material name="green">
-            <color rgba="0 0.9 0.3 1" />
-        </material>
-        <material name="white">
-            <color rgba="1 1 1 1" />
-        </material>
         <!--Main gripper-->
         <link name="${prefix}schunk_egp40_body_link">
@@ -33,5 +24,4 @@
                 </geometry>
                 <origin rpy="${pi/2} 0 0" xyz="${-body_length/2} ${body_width/2} ${-body_height/2}" />
-                <material name="green" />
             </visual>
             <collision>
@@ -52,5 +42,4 @@
                 </geometry>
                 <origin rpy="${pi/2} 0 0" xyz="${-body_length/2} ${pincer_width/2} ${-body_height-pincer_height/2}" />
-                <material name="white" />
             </visual>
             <collision>
@@ -71,5 +60,4 @@
                 </geometry>
                 <origin rpy="${pi/2} 0 0" xyz="${-body_length/2} ${pincer_width/2} ${-body_height-pincer_height/2}" />
-                <material name="blue" />
             </visual>
             <collision>
