Commit message: new description package has been created for flange

File: schunk_egp40_description/urdf/schunk_egp40.urdf (robot description, URDF)
Before this commit: robot schunk_egp40, 6 links, 5 joints
Links:
- removed link schunk_egp40_base_link

File: schunk_egp40_description/urdf/schunk_egp40.xacro (robot description, xacro)
@@ -26,20 +26,4 @@
             <color rgba="1 1 1 1" />
         </material>
-        <!--Base plate-->
-        <link name="${prefix}schunk_egp40_base_link">
-            <visual>
-                <geometry>
-                    <mesh filename="package://prbt_cell_description/meshes/flange_v3.STL" scale="0.001 0.001 0.001" />
-                </geometry>
-                <material name="blue" />
-                <origin rpy="${pi} 0 0" xyz="-${base_diameter/2} ${base_diameter/2} ${base_height}" />
-            </visual>
-            <collision>
-                <geometry>
-                    <mesh filename="package://prbt_cell_description/meshes/flange_v3.STL" scale="0.001 0.001 0.001" />
-                </geometry>
-                <origin rpy="${pi} 0 0" xyz="-${base_diameter/2} ${base_diameter/2} ${base_height}" />
-            </collision>
-        </link>
         <!--Main gripper-->
         <link name="${prefix}schunk_egp40_body_link">

Commit message: fix mesh package path

File: schunk_egp40_description/urdf/schunk_egp40.urdf (robot description, URDF)
Before this commit: robot schunk_egp40, 5 links, 5 joints
Links:
- link schunk_egp40_body_link: geometry collision mesh filename=package://schunk_egp40_description/meshes/schunk_egp40_body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 scale=0.001 0.001 0.001; visual mesh filename=package://schunk_egp40_description/meshes/schunk_egp40_body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 scale=0.001 0.001 0.001
- link schunk_egp40_finger_left_link: geometry collision mesh filename=package://schunk_egp40_description/meshes/schunk_finger_lef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 scale=0.001 0.001 0.001; visual mesh filename=package://schunk_egp40_description/meshes/schunk_finger_lef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 scale=0.001 0.001 0.001
- link schunk_egp40_finger_right_link: geometry collision mesh filename=package://schunk_egp40_description/meshes/schunk_finger_rig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 scale=0.001 0.001 0.001; visual mesh filename=package://schunk_egp40_description/meshes/schunk_finger_rig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 scale=0.001 0.001 0.001

File: schunk_egp40_description/urdf/schunk_egp40.xacro (robot description, xacro)
@@ -21,5 +21,5 @@
             <visual>
                 <geometry>
-                    <mesh filename="package://prbt_cell_description/meshes/schunk_egp40_body.STL" scale="0.001 0.001 0.001" />
+                    <mesh filename="package://schunk_egp40_description/meshes/schunk_egp40_body.STL" scale="0.001 0.001 0.001" />
                 </geometry>
                 <origin rpy="${pi/2} 0 0" xyz="${-body_length/2} ${body_width/2} ${-body_height/2}" />
@@ -27,5 +27,5 @@
             <collision>
                 <geometry>
-                    <mesh filename="package://prbt_cell_description/meshes/schunk_egp40_body.STL" scale="0.001 0.001 0.001" />
+                    <mesh filename="package://schunk_egp40_description/meshes/schunk_egp40_body.STL" scale="0.001 0.001 0.001" />
                 </geometry>
                 <origin rpy="${pi/2} 0 0" xyz="${-body_length/2} ${body_width/2} ${-body_height/2}" />
@@ -39,5 +39,5 @@
             <visual>
                 <geometry>
-                    <mesh filename="package://prbt_cell_description/meshes/schunk_finger_left.STL" scale="0.001 0.001 0.001" />
+                    <mesh filename="package://schunk_egp40_description/meshes/schunk_finger_left.STL" scale="0.001 0.001 0.001" />
                 </geometry>
                 <origin rpy="${pi/2} 0 0" xyz="${-body_length/2} ${pincer_width/2} ${-body_height-pincer_height/2}" />
@@ -45,5 +45,5 @@
             <collision>
                 <geometry>
-                    <mesh filename="package://prbt_cell_description/meshes/schunk_finger_left.STL" scale="0.001 0.001 0.001" />
+                    <mesh filename="package://schunk_egp40_description/meshes/schunk_finger_left.STL" scale="0.001 0.001 0.001" />
                 </geometry>
                 <origin rpy="${pi/2} 0 0" xyz="${-body_length/2} ${pincer_width/2} ${-body_height-pincer_height/2}" />
@@ -57,5 +57,5 @@
             <visual>
                 <geometry>
-                    <mesh filename="package://prbt_cell_description/meshes/schunk_finger_right.STL" scale="0.001 0.001 0.001" />
+                    <mesh filename="package://schunk_egp40_description/meshes/schunk_finger_right.STL" scale="0.001 0.001 0.001" />
                 </geometry>
                 <origin rpy="${pi/2} 0 0" xyz="${-body_length/2} ${pincer_width/2} ${-body_height-pincer_height/2}" />
@@ -63,5 +63,5 @@
             <collision>
                 <geometry>
-                    <mesh filename="package://prbt_cell_description/meshes/schunk_finger_right.STL" scale="0.001 0.001 0.001" />
+                    <mesh filename="package://schunk_egp40_description/meshes/schunk_finger_right.STL" scale="0.001 0.001 0.001" />
                 </geometry>
                 <origin rpy="${pi/2} 0 0" xyz="${-body_length/2} ${pincer_width/2} ${-body_height-pincer_height/2}" />

Commit message: fix flange related links

File: schunk_egp40_description/urdf/schunk_egp40.urdf (robot description, URDF)
Before this commit: robot schunk_egp40, 5 links, 5 joints
Joints:
- removed joint schunk_egp40_body_joint
- joint schunk_egp40_base_joint: child schunk_egp40_base_link -> schunk_egp40_body_link
- joint schunk_egp40_tip_joint: parent schunk_egp40_base_link -> schunk_egp40_body_link

File: schunk_egp40_description/urdf/schunk_egp40.xacro (robot description, xacro)
@@ -74,9 +74,4 @@
         <link name="tool_tip" />
         <!-- Joints-->
-        <joint name="${prefix}schunk_egp40_body_joint" type="fixed">
-            <parent link="${prefix}schunk_egp40_base_link" />
-            <child link="${prefix}schunk_egp40_body_link" />
-            <origin xyz="0.0 0.0 ${body_height/2+base_height}" rpy="0.0 0.0 0.0" />
-        </joint>
         <joint name="${prefix}schunk_egp40_finger_left_joint" type="prismatic">
             <parent link="${prefix}schunk_egp40_body_link" />
@@ -98,5 +93,5 @@
         </joint>
         <joint name="${prefix}schunk_egp40_tip_joint" type="fixed">
-            <parent link="${prefix}schunk_egp40_base_link" />
+            <parent link="${prefix}schunk_egp40_body_link" />
             <child link="tool_tip" />
             <origin xyz="0 0 ${body_height_max}" rpy="0.0 0.0 0.0" />
@@ -107,5 +102,5 @@
         >
             <parent link="${parent}" />
-            <child link="${prefix}schunk_egp40_base_link" />
+            <child link="${prefix}schunk_egp40_body_link" />
             <xacro:insert_block name="origin" />
         </joint>

Commit message: remove world link

File: schunk_egp40_description/urdf/schunk_egp40.urdf (robot description, URDF)
Before this commit: robot schunk_egp40, 5 links, 4 joints
Links:
- removed link world
Joints:
- removed joint schunk_egp40_base_joint
